File: ATXm5v.sch (KiCad schematic (older format))
At the start: 5 parts, among them J1 ATX IN, J2 ATX OUT, U1 L7905

Commit message: Add initial pcb
Parts:
- C1, C2: footprint Capacitor_SMD:C_1206_3216Metric_Pad1.42x1.75mm_HandSolder -> Capacitor_SMD:C_1206_3216Metric_Pad1.33x1.80mm_HandSolder
- J2: footprint Connector_Molex:Molex_Mini-Fit_Jr_5569-20A2_2x10_P4.20mm_Horizontal -> ATXm5v:ATX-Edge
Changed lines of the file:
@@
 F 0 "C2" H 8750 1500 50  0000 L CNN
 F 1 "100nF" H 8750 1300 50  0000 L CNN
-F 2 "Capacitor_SMD:C_1206_3216Metric_Pad1.42x1.75mm_HandSolder" H 8700 1400 50  0001 C CNN
+F 2 "Capacitor_SMD:C_1206_3216Metric_Pad1.33x1.80mm_HandSolder" H 8700 1400 50  0001 C CNN
 F 3 "~" H 8700 1400 50  0001 C CNN
 	1    8700 1400
@@
 F 0 "C1" H 7800 1450 50  0000 L CNN
 F 1 "10uF" H 7800 1350 50  0000 L CNN
-F 2 "Capacitor_SMD:C_1206_3216Metric_Pad1.42x1.75mm_HandSolder" H 7750 1400 50  0001 C CNN
+F 2 "Capacitor_SMD:C_1206_3216Metric_Pad1.33x1.80mm_HandSolder" H 7750 1400 50  0001 C CNN
 F 3 "~" H 7750 1400 50  0001 C CNN
 	1    7750 1400
@@
 F 0 "J2" H 4850 4267 50  0000 C CNN
 F 1 "ATX OUT" H 4850 4176 50  0000 C CNN
-F 2 "Connector_Molex:Molex_Mini-Fit_Jr_5569-20A2_2x10_P4.20mm_Horizontal" H 4800 3650 50  0001 C CNN
+F 2 "ATXm5v:ATX-Edge" H 4800 3650 50  0001 C CNN
 F 3 "~" H 4800 3650 50  0001 C CNN
 	1    4800 3650
@@
 ~PS_ON
 $Comp
-L power:VCC #PWR?
+L power:VCC #PWR0101
 U 1 1 6154253F
 P 5300 4100
-F 0 "#PWR?" H 5300 3950 50  0001 C CNN
+F 0 "#PWR0101" H 5300 3950 50  0001 C CNN
 F 1 "VCC" V 5317 4228 50  0000 L CNN
 F 2 "" H 5300 4100 50  0001 C CNN
@@
 	5150 4100 5150 4150
 $Comp
-L power:VCC #PWR?
+L power:VCC #PWR0102
 U 1 1 6154254F
 P 4500 3550
-F 0 "#PWR?" H 4500 3400 50  0001 C CNN
+F 0 "#PWR0102" H 4500 3400 50  0001 C CNN
 F 1 "VCC" V 4517 3677 50  0000 L CNN
 F 2 "" H 4500 3550 50  0001 C CNN
@@
 	4500 3550 4600 3550
 $Comp
-L power:VCC #PWR?
+L power:VCC #PWR0104
 U 1 1 6154255A
 P 4500 3750
-F 0 "#PWR?" H 4500 3600 50  0001 C CNN
+F 0 "#PWR0104" H 4500 3600 50  0001 C CNN
 F 1 "VCC" V 4517 3877 50  0000 L CNN
 F 2 "" H 4500 3750 50  0001 C CNN
@@
 +12V
 $Comp
-L power:GND #PWR?
+L power:GND #PWR0105
 U 1 1 61542569
 P 3850 3650
-F 0 "#PWR?" H 3850 3400 50  0001 C CNN
+F 0 "#PWR0105" H 3850 3400 50  0001 C CNN
 F 1 "GND" V 3855 3522 50  0000 R CNN
 F 2 "" H 3850 3650 50  0001 C CNN
@@
 	4050 3850 4050 3650
 $Comp
-L power:GND #PWR?
+L power:GND #PWR0106
 U 1 1 6154257A
 P 6000 3650
-F 0 "#PWR?" H 6000 3400 50  0001 C CNN
+F 0 "#PWR0106" H 6000 3400 50  0001 C CNN
 F 1 "GND" V 6005 3522 50  0000 R CNN
 F 2 "" H 6000 3650 50  0001 C CNN
