File: ATXm5v.kicad_pcb (KiCad board)
At the start: 4 copper layers, 48.3 x 44.5 mm, 5 parts, among them J1 ATX IN, J2 ATX OUT, U1 L7905

Commit message: First revision of the board
Routing:
- net /3.3V: track 38.9 -> 75.6 mm
- net VCC: track 175.1 -> 192.9 mm, vias 2 -> 3
- net GND: track 178.2 -> 186.5 mm, vias 3 -> 4
- added copper zone on B.Cu, net GND
- added copper zone on F.Cu, net GND
- added copper zone on In1.Cu, net GND
- added copper zone on In2.Cu, net GND
Changed lines of the file:
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@@
     (thickness 1.6)
     (drawings 8)
-    (tracks 101)
+    (tracks 117)
     (zones 0)
     (modules 5)
@@
   )
   (setup
-    (last_trace_width 2)
+    (last_trace_width 1)
     (user_trace_width 0.4)
     (user_trace_width 0.6)
@@
     (uvia_dia 0.3)
     (uvia_drill 0.1)
-    (add_net /3.3V)
-    (add_net /5VSB)
     (add_net /PWR_OK)
     (add_net /~PS_ON)
@@
     (uvia_drill 0.1)
     (add_net /+12V)
+    (add_net /3.3V)
     (add_net GND)
     (add_net VCC)
@@
     (add_net /-12V)
     (add_net /-5V)
+    (add_net /5VSB)
   )
   (module Capacitor_SMD:C_1206_3216Metric_Pad1.33x1.80mm_HandSolder (layer F.Cu)
@@
     (tags "D2PAK DDPAK TO-263 D2PAK-3 TO-263-3 SOT-404")
     (attr smd)
-    (fp_text reference U1 (at 0 -6.65) (layer F.SilkS)
+    (fp_text reference U1 (at -5.08 -5.08) (layer F.SilkS)
       (effects (font (size 1 1) (thickness 0.15)))
     )
@@
   (module ATXm5v:ATX-Edge (layer F.Cu)
     (at 128.27 77.47)
-    (fp_text reference J2 (at 0 -3.556) (layer F.SilkS)
+    (fp_text reference J2 (at -2.54 0 90) (layer F.SilkS)
       (effects (font (size 1 1) (thickness 0.15)))
     )
@@
   (segment (start 149.27 66.63) (end 149.27 66.72) (width 2) (layer B.Cu) (net 1))
   (segment (start 153.47 70.92) (end 153.47 77.47) (width 2) (layer B.Cu) (net 1))
-  (segment (start 153.47 52.49) (end 153.47 70.92) (width 2) (layer B.Cu) (net 1))
+  (segment (start 153.47 59.49) (end 158.55 59.49) (width 1) (layer B.Cu) (net 1))
+  (segment (start 153.47 52.49) (end 153.47 59.49) (width 2) (layer B.Cu) (net 1))
+  (segment (start 153.47 59.49) (end 153.47 70.92) (width 2) (layer B.Cu) (net 1))
+  (via (at 159.72 62.23) (size 1.5) (drill 0.6) (layers F.Cu B.Cu) (net 1))
+  (segment (start 159.72 60.66) (end 159.72 62.23) (width 1) (layer B.Cu) (net 1))
+  (segment (start 158.55 59.49) (end 159.72 60.66) (width 1) (layer B.Cu) (net 1))
   (segment (start 163.92001 53.839141) (end 163.92001 49.04001) (width 0.6) (layer F.Cu) (net 2))
   (segment (start 161.87 55.889151) (end 163.92001 53.839141) (width 0.6) (layer F.Cu) (net 2))
   (segment (start 163.92001 49.04001) (end 161.87 46.99) (width 0.6) (layer F.Cu) (net 2))
   (segment (start 161.87 77.47) (end 161.87 55.889151) (width 0.6) (layer F.Cu) (net 2))
-  (segment (start 166.07 52.49) (end 166.07 77.47) (width 2) (layer B.Cu) (net 3))
   (segment (start 161.87 52.49) (end 161.87 77.47) (width 2) (layer B.Cu) (net 3))
-  (segment (start 161.87 52.49) (end 166.07 52.49) (width 2) (layer B.Cu) (net 3))
   (segment (start 140.87 46.800899) (end 140.87 46.99) (width 2) (layer In1.Cu) (net 3))
   (segment (start 143.930909 43.73999) (end 140.87 46.800899) (width 2) (layer In1.Cu) (net 3))
@@
   (segment (start 149.27 73.07) (end 148.59 72.39) (width 2) (layer F.Cu) (net 3))
   (segment (start 149.27 77.47) (end 149.27 73.07) (width 2) (layer F.Cu) (net 3))
+  (via (at 166.07 71.42) (size 1.5) (drill 0.6) (layers F.Cu B.Cu) (net 3))
+  (segment (start 165.1 72.39) (end 166.07 71.42) (width 2) (layer In1.Cu) (net 3))
+  (segment (start 148.59 72.39) (end 165.1 72.39) (width 2) (layer In1.Cu) (net 3))
+  (segment (start 166.07 71.42) (end 166.07 77.47) (width 2) (layer B.Cu) (net 3))
+  (segment (start 166.07 71.42) (end 166.07 52.49) (width 2) (layer In1.Cu) (net 3))
+  (segment (start 166.07 52.49) (end 161.87 52.49) (width 2) (layer In1.Cu) (net 3))
   (via (at 128.27 77.47) (size 1.5) (drill 0.6) (layers F.Cu B.Cu) (net 9))
   (segment (start 132.47 56.5625) (end 133.0575 57.15) (width 1) (layer F.Cu) (net 4))
@@
   (segment (start 159.52001 53.83999) (end 157.67 55.69) (width 0.6) (layer F.Cu) (net 8))
   (segment (start 132.47 77.47) (end 128.27 77.47) (width 2.5) (layer F.Cu) (net 9))
-  (segment (start 132.47 46.99) (end 128.27 46.99) (width 2) (layer In2.Cu) (net 9))
-  (segment (start 128.27 46.99) (end 128.27 52.49) (width 2) (layer In2.Cu) (net 9))
-  (segment (start 128.27 52.49) (end 128.27 77.47) (width 2) (layer In2.Cu) (net 9))
-  (zone (net 3) (net_name VCC) (layer F.Mask) (hatch edge 0.508)
+  (segment (start 132.47 46.99) (end 128.27 46.99) (width 2) (layer F.Cu) (net 9))
+  (segment (start 128.27 46.99) (end 128.27 52.49) (width 2) (layer F.Cu) (net 9))
+  (segment (start 128.27 52.49) (end 128.27 77.47) (width 2) (layer B.Cu) (net 9))
+  (segment (start 128.27 77.47) (end 127 77.47) (width 2) (layer In2.Cu) (net 9))
+  (segment (start 127 77.47) (end 125.73 76.2) (width 2) (layer In2.Cu) (net 9))
+  (segment (start 125.73 49.53) (end 128.27 46.99) (width 2) (layer In2.Cu) (net 9))
+  (segment (start 127.85 52.49) (end 125.73 54.61) (width 2) (layer In2.Cu) (net 9))
+  (segment (start 128.27 52.49) (end 127.85 52.49) (width 2) (layer In2.Cu) (net 9))
+  (segment (start 125.73 54.61) (end 125.73 49.53) (width 2) (layer In2.Cu) (net 9))
+  (segment (start 125.73 76.2) (end 125.73 54.61) (width 2) (layer In2.Cu) (net 9))
+  (zone (net 0) (net_name "") (layer F.Mask) (hatch edge 0.508)
     (connect_pads (clearance 0.508))
     (min_thickness 0.254)
@@
       )
     )
+  )
+  (zone (net 1) (net_name GND) (layer In1.Cu) (hatch edge 0.508)
+    (connect_pads (clearance 0.508))
+    (min_thickness 0.254)
+    (fill yes (arc_segments 32) (thermal_gap 0.508) (thermal_bridge_width 0.508))
+    (polygon
+      (pts
+        (xy 172.72 82.55) (xy 121.92 82.55) (xy 121.92 34.29) (xy 172.72 34.29)
+      )
+    )
+  )
+  (zone (net 1) (net_name GND) (layer In2.Cu) (hatch edge 0.508)
+    (connect_pads (clearance 0.508))
+    (min_thickness 0.254)
+    (fill yes (arc_segments 32) (thermal_gap 0.508) (thermal_bridge_width 0.508))
+    (polygon
+      (pts
+        (xy 172.72 82.55) (xy 121.92 82.55) (xy 121.92 34.29) (xy 172.72 34.29)
+      )
+    )
+  )
+  (zone (net 1) (net_name GND) (layer B.Cu) (hatch edge 0.508)
+    (connect_pads (clearance 0.508))
+    (min_thickness 0.254)
+    (fill yes (arc_segments 32) (thermal_gap 0.508) (thermal_bridge_width 0.508))
+    (polygon
+      (pts
+        (xy 172.72 82.55) (xy 121.92 82.55) (xy 121.92 34.29) (xy 172.72 34.29)
+      )
+    )
+  )
+  (zone (net 1) (net_name GND) (layer F.Cu) (hatch edge 0.508)
+    (connect_pads (clearance 0.508))
+    (min_thickness 0.254)
+    (fill yes (arc_segments 32) (thermal_gap 0.508) (thermal_bridge_width 0.508))
+    (polygon
+      (pts
+        (xy 172.72 82.55) (xy 121.92 82.55) (xy 121.92 74.93) (xy 138.43 74.93) (xy 138.43 54.61)
+        (xy 121.92 54.61) (xy 121.92 34.29) (xy 172.72 34.29)
+      )
+    )
